Commit message: robot: add planar base joint and align SRDF
Introduce a planar  with intermediate  in the URDF so MoveIt treats the chassis as a 3-DoF base, and update the SRDF virtual joint parent frame to match. Wheels remain kinematically ignored while providing vx/vy/yaw control inputs.

File: mobile_arm_whole_body/urdf/arm_on_car_center_rotZ_n90_center.urdf (robot description, URDF)
Before this commit: robot chassis_with_single_arm, 9 links, 8 joints
Links:
- added link odom_link
Joints:
- added joint world_joint: type planar, parent odom_link, child chassis_center_link, origin xyz=0 0 0 rpy=0 0 0, axis 0 0 1
- added joint world_to_odom: type fixed, parent world, child odom_link, origin xyz=0 0 0 rpy=0 0 0

Commit message: bringup: load moveit params into rviz and planner
Provide MoveIt configuration parameters (robot description, semantic, kinematics, joint limits, planning pipelines) to both the RViz session and the whole_body_planner so meshes and planning scene assets load correctly. Simplify the streaming launch to reuse the MoveIt demo RViz, propagate the rviz argument, and share the configuration via MoveItConfigsBuilder. Revert the experimental URDF planar joint back to the original while keeping the SRDF robot name fix.

File: mobile_arm_whole_body/urdf/arm_on_car_center_rotZ_n90_center.urdf (robot description, URDF)
Before this commit: robot chassis_with_single_arm, 10 links, 10 joints
Links:
- removed link odom_link
Joints:
- removed joint world_joint
- removed joint world_to_odom
